File: kicad/solder_station.sch (KiCad schematic (older format))
At the start: 23 parts, among them IC1 ATMEGA8-P, Q1 Q_NMOS_GDS, Q2 Q_PMOS_DGS, U1 7805, U2 LM2902N

Commit message: Update.
Parts:
- removed U1: 7805, symbol 7805
- added CON1: AVR-ISP-6, connector:CONNECTOR 3 2, symbol AVR-ISP-6
- added P1: Weller Connector, my_footprints:ZIP-3, symbol CONN_01X03
- added U1: LM7805, TO_SOT_Packages_THT:TO-220_Neutral123_Vertical_LargePads, symbol LM_7805
- C1, C2, C3: footprint (none) -> Capacitors_ThroughHole:C_Disc_D3_P2.5
- C4, C5: value C -> 100nF; footprint (none) -> Capacitors_ThroughHole:C_Disc_D3_P2.5
- C6, C7: value C -> 10nF; footprint (none) -> Capacitors_ThroughHole:C_Disc_D3_P2.5
- DS1: renamed from DS?; footprint WC1602A -> Pin_Headers:Pin_Header_Straight_1x16
- IC1: footprint DIL28 -> Housings_DIP:DIP-28_W7.62mm_LongPads
- L1: footprint (none) -> Choke_Axial_ThroughHole:Choke_Horizontal_RM10mm
- Q1: value Q_NMOS_GDS -> BS170; footprint (none) -> TO_SOT_Packages_THT:TO-92_Inline_Wide
- Q2: value Q_PMOS_DGS -> IRF4905; footprint (none) -> TO_SOT_Packages_THT:TO-220_Neutral123_Vertical; symbol Q_PMOS_DGS -> Q_PMOS_GDS
- R1: value R -> 100kΩ; footprint (none) -> Resistors_ThroughHole:Resistor_Horizontal_RM10mm
- R2, R4, R8: value R -> 1kΩ; footprint (none) -> Resistors_ThroughHole:Resistor_Horizontal_RM10mm
- R3: value R -> 10kΩ; footprint (none) -> Resistors_ThroughHole:Resistor_Horizontal_RM10mm
- R5: footprint (none) -> Resistors_ThroughHole:Resistor_Horizontal_RM10mm
- R6: value R -> 100Ω; footprint (none) -> Resistors_ThroughHole:Resistor_Horizontal_RM10mm
- R7: value R -> 50kΩ; footprint (none) -> Resistors_ThroughHole:Resistor_Horizontal_RM10mm
- R9: renamed from R?; footprint (none) -> Resistors_ThroughHole:Resistor_Horizontal_RM10mm
- U2: footprint (none) -> TO_SOT_Packages_SMD:SOT-23-5
Connections:
- net labels added: AVcc, MISO, MOSI, RESET, SCK
- wire segments 59 -> 85
- no-connect marks 24 -> 15
Other:
- note added: "Opamp und fets noch nicht ausgesucht"
- note added: "Wert muss noch ermittelt werden"
- moved on the sheet: C4, C5

Commit message: Update schematic.
Parts:
- removed C4, C5: 100nF, Capacitors_ThroughHole:C_Disc_D3_P2.5, symbol C
- removed P1: Weller Connector, my_footprints:ZIP-3, symbol CONN_01X03
- removed U1: LM7805, TO_SOT_Packages_THT:TO-220_Neutral123_Vertical_LargePads, symbol LM_7805
- removed U2: LM2902N, TO_SOT_Packages_SMD:SOT-23-5, symbol LM2902N
- added P1: CONN_01X08, Pin_Headers:Pin_Header_Straight_1x08, symbol CONN_01X08
- added P2: CONN_01X02, Terminal_Blocks:TerminalBlock_Pheonix_MKDS1.5-2pol, symbol CONN_01X02
- added U1: LM2596_module, symbol LM2596_module
- added U2: AD8572, Housings_SOIC:SOIC-8_3.9x4.9mm_Pitch1.27mm, symbol LM358
- L1: value 10uH -> 10µH
- Q1: value BS170 -> 2N7000; symbol Q_NMOS_GDS -> Q_NMOS_DGS
- Q2: symbol Q_PMOS_GDS -> Q_NMOS_SGD
- R5: value R -> 10kΩ
Connections:
- net +5V: now also U1.3 (OUT+)
- net AVcc: now also U2.8 (V+)
- net GND: now also P1.2 (P2), P1.4 (P4), P1.5 (P5), P2.2 (P2), U1.2 (IN-), U1.4 (OUT-), U2.4 (V-)
- net at R2.1, R3.1: now also Q1.2 (G); no longer Q1.1 (G)
- net at R7.1, R8.2: now also U2.1
- net at R6.1, R7.2: now also U2.2 (-)
- net at C6.1, R4.1: now also U2.3 (+)
- net +12V: no longer names the net of Q2.2 (G)
- net +12V: now also Q1.1 (D), R5.2; no longer R5.1
- net Heater_sense renamed Sense+
- net Sense+: now also P1.3 (P3)
- net Heater_vcc renamed +24V
- net +24V: now also R5.1, P2.1 (P1), U1.1 (IN+)
- new net Heater+: P1.1 (P1), Q2.1 (S)
- no-connect marks 15 -> 18
Other:
- note added: "Belegung geraten"
- note added: "Power Input"
- note removed: "Opamp und fets noch nicht ausgesucht"
- moved on the sheet: R6

Commit message: Update kicad schematics (still incomplete).
Parts:
- added U3: EC11, symbol EC11
- IC1: value ATMEGA8-P -> ATMEGA328-P; symbol ATMEGA8-P -> ATMEGA328-P
Connections:
- net GND: now also U3.2 (C), U3.5 (E)
- net Rotary_A: now reaches IC1.24 ((PCINT9/ADC1)PC1)
- net Rotary_A: now also U3.1 (A)
- net Rotary_B: now reaches IC1.25 ((PCINT10/ADC2)PC2)
- net Rotary_B: now also U3.3 (B)
- net Button_push: now reaches IC1.26 ((PCINT11/ADC3)PC3)
- net Button_push: now also U3.4 (D)
- no-connect marks 18 -> 15
Other:
- moved on the sheet: C2, R1

Commit message: Update Schematics.
Parts:
- removed CON1: AVR-ISP-6, connector:CONNECTOR 3 2, symbol AVR-ISP-6
- removed P1: CONN_01X08, Pin_Headers:Pin_Header_Straight_1x08, symbol CONN_01X08
- added C4, C5: 22pF, Capacitors_ThroughHole:C_Disc_D3_P2.5, symbol C
- added C8: 100nF, Capacitors_ThroughHole:C_Disc_D3_P2.5, symbol C
- added P1: CONN_01X05, Pin_Headers:Pin_Header_Straight_1x05, symbol CONN_01X05
- added P3: GX16-8 Plug, symbol CONN_01X08
- added P4: UART, Pin_Headers:Pin_Header_Straight_1x03, symbol CONN_01X04
- added Y1: 16MHz, Crystals:Crystal_HC51-U_Vertical, symbol Crystal
- U1: footprint (none) -> my_footprints:LM2596
- U3: footprint (none) -> Buttons_Switches_ThroughHole:KSA_Tactile_SPST
Connections:
- net MISO is gone; now on net Rotary_A: IC1.18 ((PCINT4/MISO)PB4)
- net MOSI is gone; now on net Button_push: IC1.17 ((PCINT3/OC2A/MOSI)PB3)
- net SCK is gone; now on net Rotary_B: IC1.19 ((PCINT5/SCK)PB5)
- net Sense+ is gone; now on net Heater+: R4.2
- net Button_push: no longer IC1.26 ((PCINT11/ADC3)PC3)
- net GND: now also C4.1, C5.1, P1.1 (P1), P1.5 (P5), P3.2 (P2), P3.7 (P7), P4.2 (P2); no longer DS1.5 (R/W)
- net Heater+: now also P1.4 (P4), P3.6 (P6)
- net RESET: now also C8.2
- net Rotary_A: no longer IC1.24 ((PCINT9/ADC1)PC1)
- net Rotary_B: no longer IC1.25 ((PCINT10/ADC2)PC2)
- net at IC1.10 ((PCINT7/XTAL2/TOSC2)PB7): now also C5.2, Y1.2
- net LCD_RW: now reaches IC1.14 ((PCINT0/CLKO/ICP1)PB0)
- net LCD_RW: now also DS1.5 (R/W)
- net RX: now reaches IC1.2 ((PCINT16/RXD)PD0)
- net RX: now also P4.3 (P3)
- net TX: now reaches IC1.3 ((PCINT17/TXD)PD1)
- net TX: now also P4.4 (P4)
- net at IC1.9 ((PCINT6/XTAL1/TOSC1)PB6): now also C4.2, Y1.1
- net LDC_E renamed LCD_E
- new net Button_connected: IC1.25 ((PCINT10/ADC2)PC2), P1.3 (P3), P3.5 (P5)
- new net Button_standby: IC1.26 ((PCINT11/ADC3)PC3), P1.2 (P2), P3.4 (P4)
- new net DTR: C8.1, P4.1 (P1)
- no-connect marks 15 -> 11
Other:
- note added: "Not part of pcb"
- note removed: "Belegung geraten"
- moved on the sheet: P2

Commit message: Update Schematics.
Parts:
- added SW1: SPST, symbol SPST
Connections:
- net GND: now also P1.2 (P2), P3.4 (P4), SW1.2
- removed net Button_standby: IC1.26 ((PCINT11/ADC3)PC3), P1.2 (P2), P3.4 (P4)
- new net: IC1.26 ((PCINT11/ADC3)PC3), SW1.1
Other:
- note added: "Extern am Addon"
Changed lines of the file:
@@
 $EndComp
 $Comp
-L GND #PWR8
+L GND #PWR6
 U 1 1 566AD0E7
 P 2850 4850
-F 0 "#PWR8" H 2850 4600 50  0001 C CNN
+F 0 "#PWR6" H 2850 4600 50  0001 C CNN
 F 1 "GND" H 2850 4700 50  0000 C CNN
 F 2 "" H 2850 4850 60  0000 C CNN
@@
 $EndComp
 $Comp
-L VCC #PWR12
+L VCC #PWR10
 U 1 1 566AD184
 P 3950 2200
-F 0 "#PWR12" H 3950 2050 50  0001 C CNN
+F 0 "#PWR10" H 3950 2050 50  0001 C CNN
 F 1 "VCC" H 3950 2350 50  0000 C CNN
 F 2 "" H 3950 2200 60  0000 C CNN
@@
 	3050 2300 4050 2300
 $Comp
-L GND #PWR18
+L GND #PWR16
 U 1 1 566AD5B2
 P 4500 2300
-F 0 "#PWR18" H 4500 2050 50  0001 C CNN
+F 0 "#PWR16" H 4500 2050 50  0001 C CNN
 F 1 "GND" H 4500 2150 50  0000 C CNN
 F 2 "" H 4500 2300 60  0000 C CNN
@@
 	2400 2750 2400 3250
 $Comp
-L GND #PWR7
+L GND #PWR5
 U 1 1 566AD654
 P 2350 2850
-F 0 "#PWR7" H 2350 2600 50  0001 C CNN
+F 0 "#PWR5" H 2350 2600 50  0001 C CNN
 F 1 "GND" H 2350 2700 50  0000 C CNN
 F 2 "" H 2350 2850 60  0000 C CNN
@@
 Connection ~ 2400 2850
 $Comp
-L VCC #PWR10
+L VCC #PWR8
 U 1 1 566AD6B9
 P 2900 2000
-F 0 "#PWR10" H 2900 1850 50  0001 C CNN
+F 0 "#PWR8" H 2900 1850 50  0001 C CNN
 F 1 "VCC" H 2900 2150 50  0000 C CNN
 F 2 "" H 2900 2000 60  0000 C CNN
@@
 	7800 3050 8000 3050
 $Comp
-L GND #PWR28
+L GND #PWR26
 U 1 1 566AFDB2
 P 8300 3500
-F 0 "#PWR28" H 8300 3250 50  0001 C CNN
+F 0 "#PWR26" H 8300 3250 50  0001 C CNN
 F 1 "GND" H 8300 3350 50  0000 C CNN
 F 2 "" H 8300 3500 60  0000 C CNN
@@
 Connection ~ 8300 3400
 $Comp
-L +24V #PWR31
+L +24V #PWR29
 U 1 1 566B014A
 P 9100 1550
-F 0 "#PWR31" H 9100 1400 50  0001 C CNN
+F 0 "#PWR29" H 9100 1400 50  0001 C CNN
 F 1 "+24V" H 9100 1690 50  0000 C CNN
 F 2 "" H 9100 1550 60  0000 C CNN
@@
 Connection ~ 8300 2250
 $Comp
-L GND #PWR30
+L GND #PWR28
 U 1 1 566AFE7A
 P 9050 6000
-F 0 "#PWR30" H 9050 5750 50  0001 C CNN
+F 0 "#PWR28" H 9050 5750 50  0001 C CNN
 F 1 "GND" H 9050 5850 50  0000 C CNN
 F 2 "" H 9050 6000 60  0000 C CNN
@@
 $EndComp
 $Comp
-L GND #PWR29
+L GND #PWR27
 U 1 1 566B0E6D
 P 8350 5500
-F 0 "#PWR29" H 8350 5250 50  0001 C CNN
+F 0 "#PWR27" H 8350 5250 50  0001 C CNN
 F 1 "GND" H 8350 5350 50  0000 C CNN
 F 2 "" H 8350 5500 60  0000 C CNN
@@
 $EndComp
 $Comp
-L GND #PWR33
+L GND #PWR32
 U 1 1 566B0EB7
 P 10200 5550
-F 0 "#PWR33" H 10200 5300 50  0001 C CNN
+F 0 "#PWR32" H 10200 5300 50  0001 C CNN
 F 1 "GND" H 10200 5400 50  0000 C CNN
 F 2 "" H 10200 5550 60  0000 C CNN
@@
 $EndComp
 $Comp
-L GND #PWR13
+L GND #PWR11
 U 1 1 566B287E
 P 4000 6800
-F 0 "#PWR13" H 4000 6550 50  0001 C CNN
+F 0 "#PWR11" H 4000 6550 50  0001 C CNN
 F 1 "GND" H 4000 6650 50  0000 C CNN
 F 2 "" H 4000 6800 60  0000 C CNN
@@
 $EndComp
 $Comp
-L GND #PWR16
+L GND #PWR14
 U 1 1 566B28D2
 P 4200 6800
-F 0 "#PWR16" H 4200 6550 50  0001 C CNN
+F 0 "#PWR14" H 4200 6550 50  0001 C CNN
 F 1 "GND" H 4200 6650 50  0000 C CNN
 F 2 "" H 4200 6800 60  0000 C CNN
@@
 	4200 6700 4200 6800
 $Comp
-L VCC #PWR14
+L VCC #PWR12
 U 1 1 566B2AEC
 P 4100 7050
-F 0 "#PWR14" H 4100 6900 50  0001 C CNN
+F 0 "#PWR12" H 4100 6900 50  0001 C CNN
 F 1 "VCC" H 4100 7200 50  0000 C CNN
 F 2 "" H 4100 7050 60  0000 C CNN
@@
 	5300 6700 5300 7000
 $Comp
-L GND #PWR21
+L GND #PWR19
 U 1 1 566B2F57
 P 5500 7000
-F 0 "#PWR21" H 5500 6750 50  0001 C CNN
+F 0 "#PWR19" H 5500 6750 50  0001 C CNN
 F 1 "GND" H 5500 6850 50  0000 C CNN
 F 2 "" H 5500 7000 60  0000 C CNN
@@
 $EndComp
 $Comp
-L VCC #PWR19
+L VCC #PWR17
 U 1 1 566B2FA4
 P 5400 7300
-F 0 "#PWR19" H 5400 7150 50  0001 C CNN
+F 0 "#PWR17" H 5400 7150 50  0001 C CNN
 F 1 "VCC" H 5400 7450 50  0000 C CNN
 F 2 "" H 5400 7300 60  0000 C CNN
@@
 $EndComp
 $Comp
-L +24V #PWR27
+L +24V #PWR25
 U 1 1 566DD4CA
 P 7650 900
-F 0 "#PWR27" H 7650 750 50  0001 C CNN
+F 0 "#PWR25" H 7650 750 50  0001 C CNN
 F 1 "+24V" H 7650 1040 50  0000 C CNN
 F 2 "" H 7650 900 60  0000 C CNN
@@
 $EndComp
 $Comp
-L GND #PWR26
+L GND #PWR24
 U 1 1 566DD545
 P 7550 800
-F 0 "#PWR26" H 7550 550 50  0001 C CNN
+F 0 "#PWR24" H 7550 550 50  0001 C CNN
 F 1 "GND" H 7550 650 50  0000 C CNN
 F 2 "" H 7550 800 60  0000 C CNN
@@
 $EndComp
 $Comp
-L GND #PWR15
+L GND #PWR13
 U 1 1 56874984
 P 4150 1100
-F 0 "#PWR15" H 4150 850 50  0001 C CNN
+F 0 "#PWR13" H 4150 850 50  0001 C CNN
 F 1 "GND" H 4150 950 50  0000 C CNN
 F 2 "" H 4150 1100 60  0000 C CNN
@@
 $EndComp
 $Comp
-L GND #PWR11
+L GND #PWR9
 U 1 1 568749D7
 P 3250 1100
-F 0 "#PWR11" H 3250 850 50  0001 C CNN
+F 0 "#PWR9" H 3250 850 50  0001 C CNN
 F 1 "GND" H 3250 950 50  0000 C CNN
 F 2 "" H 3250 1100 60  0000 C CNN
@@
 $EndComp
 $Comp
-L +24V #PWR9
+L +24V #PWR7
 U 1 1 56874A72
 P 2900 1000
-F 0 "#PWR9" H 2900 850 50  0001 C CNN
+F 0 "#PWR7" H 2900 850 50  0001 C CNN
 F 1 "+24V" H 2900 1140 50  0000 C CNN
 F 2 "" H 2900 1000 60  0000 C CNN
@@
 	2900 1000 3250 1000
 $Comp
-L +5V #PWR17
+L +5V #PWR15
 U 1 1 56874C19
 P 4400 1000
-F 0 "#PWR17" H 4400 850 50  0001 C CNN
+F 0 "#PWR15" H 4400 850 50  0001 C CNN
 F 1 "+5V" H 4400 1140 50  0000 C CNN
 F 2 "" H 4400 1000 60  0000 C CNN
@@
 Connection ~ 3950 2300
 $Comp
-L VCC #PWR22
+L VCC #PWR20
 U 1 1 56A13B2D
 P 5900 4600
-F 0 "#PWR22" H 5900 4450 50  0001 C CNN
+F 0 "#PWR20" H 5900 4450 50  0001 C CNN
 F 1 "VCC" H 5900 4750 50  0000 C CNN
 F 2 "" H 5900 4600 60  0000 C CNN
@@
 	5300 1800 5500 1800
 $Comp
-L GND #PWR23
+L GND #PWR21
 U 1 1 56A15474
 P 6150 1750
-F 0 "#PWR23" H 6150 1500 50  0001 C CNN
+F 0 "#PWR21" H 6150 1500 50  0001 C CNN
 F 1 "GND" H 6150 1600 50  0000 C CNN
 F 2 "" H 6150 1750 60  0000 C CNN
@@
 $EndComp
 $Comp
-L GND #PWR20
+L GND #PWR18
 U 1 1 56A154CA
 P 5450 1700
-F 0 "#PWR20" H 5450 1450 50  0001 C CNN
+F 0 "#PWR18" H 5450 1450 50  0001 C CNN
 F 1 "GND" H 5450 1550 50  0000 C CNN
 F 2 "" H 5450 1700 60  0000 C CNN
@@
 	10650 1300 9950 1300
 $Comp
-L GND #PWR34
+L GND #PWR33
 U 1 1 56A3D831
 P 11000 1450
-F 0 "#PWR34" H 11000 1200 50  0001 C CNN
+F 0 "#PWR33" H 11000 1200 50  0001 C CNN
 F 1 "GND" H 11000 1300 50  0000 C CNN
 F 2 "" H 11000 1450 60  0000 C CNN
@@
 	0    -1   -1   0
 $EndComp
-Text GLabel 5100 3800 2    60   Input ~ 0
+Text GLabel 6250 3800 2    60   Input ~ 0
 Button_standby
 Text GLabel 5100 3700 2    60   Input ~ 0
@@
 Connection ~ 10250 1450
 $Comp
-L GND #PWR32
+L GND #PWR30
 U 1 1 56A3ED56
 P 9250 700
-F 0 "#PWR32" H 9250 450 50  0001 C CNN
+F 0 "#PWR30" H 9250 450 50  0001 C CNN
 F 1 "GND" H 9250 550 50  0000 C CNN
 F 2 "" H 9250 700 60  0000 C CNN
@@
 Connection ~ 5800 3100
 $Comp
-L GND #PWR24
+L GND #PWR22
 U 1 1 56A4108C
 P 6500 3250
-F 0 "#PWR24" H 6500 3000 50  0001 C CNN
+F 0 "#PWR22" H 6500 3000 50  0001 C CNN
 F 1 "GND" H 6500 3100 50  0000 C CNN
 F 2 "" H 6500 3250 60  0000 C CNN
@@
 TX
 $Comp
-L GND #PWR25
+L GND #PWR23
 U 1 1 56A42505
 P 6600 5500
-F 0 "#PWR25" H 6600 5250 50  0001 C CNN
+F 0 "#PWR23" H 6600 5250 50  0001 C CNN
 F 1 "GND" H 6600 5350 50  0000 C CNN
 F 2 "" H 6600 5500 60  0000 C CNN
@@
 	5100 3700 4950 3700
 Wire Wire Line
-	5100 3800 4950 3800
+	4950 3800 5150 3800
+$Comp
+L GND #PWR31
+U 1 1 56A4FE40
+P 10000 1000
+F 0 "#PWR31" H 10000 750 50  0001 C CNN
+F 1 "GND" H 10000 850 50  0000 C CNN
+F 2 "" H 10000 1000 60  0000 C CNN
+F 3 "" H 10000 1000 60  0000 C CNN
+	1    10000 1000
+	-1   0    0    1
+$EndComp
+Wire Wire Line
+	10000 1000 10000 1150
+Connection ~ 10000 1150
+$Comp
+L SPST SW1
+U 1 1 56A4FF92
+P 5650 3800
+F 0 "SW1" H 5550 3900 50  0000 C CNN
+F 1 "SPST" H 5950 3900 50  0000 C CNN
+F 2 "" H 5650 3800 60  0000 C CNN
+F 3 "" H 5650 3800 60  0000 C CNN
+	1    5650 3800
+	1    0    0    1
+$EndComp
+Wire Wire Line
+	6150 3800 6250 3800
+Text Notes 5400 4000 0    60   ~ 0
+Extern am Addon
 $EndSCHEMATC
