File: kicad/solder_station.sch (KiCad schematic (older format))
At the start: 64 parts, among them IC1 ATMEGA328-P, P1 CONN_01X05, P2 CONN_01X02, P3 Standby, P4 UART, P5 12V_Out, Q1 2N7000, Q2 IRF4905, U1 LM2596_module, U2 AD8572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

Commit message: [Kicad] Small updates
Parts:
- C15, C24: value 1mF -> 470µF
- C9: footprint Capacitors_ThroughHole:C_Radial_D13_L21_P5 -> Capacitors_ThroughHole:C_Radial_D10_L25_P5
- P1: footprint Terminal_Blocks:TerminalBlock_Pheonix_PT-3.5mm_5pol -> Terminal_Blocks:TerminalBlock_Pheonix_MKDS1.5-5pol
- P2: footprint Terminal_Blocks:TerminalBlock_Pheonix_PT-3.5mm_2pol -> Terminal_Blocks:TerminalBlock_Pheonix_MKDS1.5-2pol
- R8: value 1kΩ -> 6.7kΩ
- U2: symbol LM293 -> LM293-RESCUE-solder_station
Connections:
- net Heater+: no longer C6.1
- net at D1.1 (K), D2.2 (A), R4.1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: now also C6.1
Other:
- moved on the sheet: C6, C9, D4, R4
