File: kicad/solder_station.kicad_pcb (KiCad board)
At the start: 2 copper layers, 63.8 x 64 mm, 69 parts, among them IC1 ATMEGA328-P, P1 CONN_01X05, P2 CONN_01X02, P3 Standby, P4 UART, P5 12V_Out, Q1 2N7000, Q2 IRF4905, U1 LM2596_module, U2 AD8572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

Commit message: [Kicad] Small updates
Parts:
- C15, C24: value 1mF -> 470µF
- C9: footprint Capacitors_ThroughHole:C_Radial_D13_L21_P5 -> Capacitors_ThroughHole:C_Radial_D10_L25_P5
- P1: footprint Terminal_Blocks:TerminalBlock_Pheonix_PT-3.5mm_5pol -> Terminal_Blocks:TerminalBlock_Pheonix_MKDS1.5-5pol
- P2: footprint Terminal_Blocks:TerminalBlock_Pheonix_PT-3.5mm_2pol -> Terminal_Blocks:TerminalBlock_Pheonix_MKDS1.5-2pol
- R8: value 1kΩ -> 6.7kΩ
- moved C6 9.90 mm to (149.4, 112.2), turned to 270 degrees
- moved P1 3.30 mm to (129.9, 123.9)
- moved R11 3.16 mm to (132.4, 121.0)
- moved C7 3.04 mm to (148.3, 99.6)
- moved C15 1.94 mm to (134.4, 106.4), turned to 0 degrees
- moved C9 1.00 mm to (107.0, 120.8)
- moved P2 0.89 mm to (119.7, 123.9)
- moved Q2 0.81 mm to (128.2, 113.2)
- moved Q1 0.75 mm to (131.1, 105.2)
- moved C24 0.65 mm to (133.7, 113.4)
Connections:
- C6 pad 1: /Heater+ -> Net-(C6-Pad1)
- D1 pad 1: Net-(D1-Pad1) -> Net-(C6-Pad1)
- D2 pad 2: Net-(D1-Pad1) -> Net-(C6-Pad1)
- R4 pad 1: Net-(D1-Pad1) -> Net-(C6-Pad1)
- U2 pad 3: Net-(D1-Pad1) -> Net-(C6-Pad1)
Routing:
- net Net-(C6-Pad1): track 0.00 -> 21.2 mm
- net Net-(D1-Pad1): track 18.1 -> 0.00 mm
- net +24V: track 57.5 -> 49.7 mm
- net /Button_connected: track 55.6 -> 51.2 mm
- net /Tip: track 2.42 -> 3.52 mm
- net /Heater+: track 28.4 -> 27.3 mm
- net Net-(Q1-Pad2): track 7.97 -> 8.49 mm
